File: hardware/peripheral/p2x3p-001.brd (EAGLE design)
At the start: 18 x 31 mm, 5 parts

Commit message: WIP.
Parts:
- added C1, C2: (no value), rcl:C025-024X044
- moved LOGO1 12.5 mm to (2.75, 28.0), flipped to the top, turned to 0 degrees
Connections:
- net ANLG0: now also J1.1
- net ANLG1: now also J2.1
- net GND: now also C1.2, C2.2, J1.2, J2.2
- net VCC: now also C1.1, C2.1, J1.3, J2.3
Routing:
- net GND: track 0.00 -> 36.0 mm
- net VCC: track 0.00 -> 28.4 mm
- net ANLG0: track 0.00 -> 13.4 mm
- net ANLG1: track 0.00 -> 11.1 mm
Other:
- board text added: "3P Connertors 0.0.1-X"
- board text removed: "Hex Sw 0.0.1-X"
