File: hardware/peripheral/p2x3p-001.brd (EAGLE design)
At the start: 18 x 31 mm, 7 parts

Commit message: Silk.
Parts:
- renumbered J1 to J31, J2 to J32, JP1 to SV1
Changed lines of the file:
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@@
 <elements>
 <element name="LOGO1" library="SparkFun-Aesthetics" package="OSHW-LOGO-S_COPPER" value="OSHW-LOGOS-COPPER" x="2.75" y="28" smashed="yes"/>
-<element name="JP1" library="pinhead" library_urn="urn:adsk.eagle:library:325" package="2X08" package3d_urn="urn:adsk.eagle:package:22481/2" value="" x="13" y="15.5" smashed="yes" rot="R90">
+<element name="SV1" library="pinhead" library_urn="urn:adsk.eagle:library:325" package="2X08" package3d_urn="urn:adsk.eagle:package:22481/2" value="" x="13" y="15.5" smashed="yes" rot="R90">
 <attribute name="NAME" x="9.5" y="15.5" size="1" layer="25" ratio="10" rot="R90" align="center"/>
 <attribute name="POPULARITY" value="6" x="13" y="15.5" size="1.778" layer="27" rot="R90" display="off"/>
@@
 </element>
 <element name="U$1" library="pineapple" package="PINEAPPLE450_SILK" value="PINEAPPLE450_SILK" x="0.5" y="21" smashed="yes" rot="MR90"/>
-<element name="J1" library="SparkFun-Connectors" library_urn="urn:adsk.eagle:library:513" package="JST-3-PTH" package3d_urn="urn:adsk.eagle:package:38069/1" value="" x="6" y="21" smashed="yes" rot="R90">
+<element name="J31" library="SparkFun-Connectors" library_urn="urn:adsk.eagle:library:513" package="JST-3-PTH" package3d_urn="urn:adsk.eagle:package:38069/1" value="" x="6" y="21" smashed="yes" rot="R90">
 <attribute name="NAME" x="4" y="26" size="1" layer="25" ratio="20" align="center"/>
 <attribute name="PROD_ID" value="WIRE-10037" x="6" y="21" size="1.778" layer="27" rot="R90" display="off"/>
@@
 <attribute name="VALUE" x="3.46" y="19.349" size="0.6096" layer="27" font="vector" ratio="20" rot="R90"/>
 </element>
-<element name="J2" library="SparkFun-Connectors" library_urn="urn:adsk.eagle:library:513" package="JST-3-PTH" package3d_urn="urn:adsk.eagle:package:38069/1" value="" x="6" y="10" smashed="yes" rot="R90">
+<element name="J32" library="SparkFun-Connectors" library_urn="urn:adsk.eagle:library:513" package="JST-3-PTH" package3d_urn="urn:adsk.eagle:package:38069/1" value="" x="6" y="10" smashed="yes" rot="R90">
 <attribute name="NAME" x="4" y="5" size="1" layer="25" ratio="20" align="center"/>
 <attribute name="PROD_ID" value="WIRE-10037" x="6" y="10" size="1.778" layer="27" rot="R90" display="off"/>
@@
 <signals>
 <signal name="GND">
-<contactref element="JP1" pad="1"/>
-<contactref element="JP1" pad="5"/>
-<contactref element="JP1" pad="9"/>
-<contactref element="JP1" pad="13"/>
-<contactref element="J1" pad="2"/>
-<contactref element="J2" pad="2"/>
+<contactref element="SV1" pad="1"/>
+<contactref element="SV1" pad="5"/>
+<contactref element="SV1" pad="9"/>
+<contactref element="SV1" pad="13"/>
+<contactref element="J31" pad="2"/>
+<contactref element="J32" pad="2"/>
 <contactref element="C1" pad="2"/>
 <contactref element="C2" pad="2"/>
@@
 </signal>
 <signal name="DTCT0">
-<contactref element="JP1" pad="2"/>
+<contactref element="SV1" pad="2"/>
 </signal>
 <signal name="VCC">
-<contactref element="JP1" pad="4"/>
-<contactref element="JP1" pad="16"/>
-<contactref element="JP1" pad="12"/>
-<contactref element="JP1" pad="8"/>
-<contactref element="J1" pad="3"/>
-<contactref element="J2" pad="3"/>
+<contactref element="SV1" pad="4"/>
+<contactref element="SV1" pad="16"/>
+<contactref element="SV1" pad="12"/>
+<contactref element="SV1" pad="8"/>
+<contactref element="J31" pad="3"/>
+<contactref element="J32" pad="3"/>
 <contactref element="C1" pad="1"/>
 <contactref element="C2" pad="1"/>
@@
 </signal>
 <signal name="DTCT1">
-<contactref element="JP1" pad="6"/>
+<contactref element="SV1" pad="6"/>
 </signal>
 <signal name="DTCT2">
-<contactref element="JP1" pad="10"/>
+<contactref element="SV1" pad="10"/>
 </signal>
 <signal name="DTCT3">
-<contactref element="JP1" pad="14"/>
+<contactref element="SV1" pad="14"/>
 </signal>
 <signal name="ANLG0">
-<contactref element="JP1" pad="3"/>
-<contactref element="J1" pad="1"/>
+<contactref element="SV1" pad="3"/>
+<contactref element="J31" pad="1"/>
 <wire x1="14.1732" y1="10.3632" x2="14.1732" y2="9.2964" width="0.1524" layer="16"/>
 <wire x1="12.8016" y1="11.7348" x2="14.1732" y2="10.3632" width="0.1524" layer="16"/>
@@
 </signal>
 <signal name="ANLG1">
-<contactref element="JP1" pad="7"/>
-<contactref element="J2" pad="1"/>
+<contactref element="SV1" pad="7"/>
+<contactref element="J32" pad="1"/>
 <wire x1="13.1064" y1="14.1732" x2="14.1732" y2="14.1732" width="0.1524" layer="1"/>
 <wire x1="11.7348" y1="12.8016" x2="13.1064" y2="14.1732" width="0.1524" layer="1"/>
@@
 </signal>
 <signal name="ANLG3">
-<contactref element="JP1" pad="15"/>
+<contactref element="SV1" pad="15"/>
 </signal>
 <signal name="ANLG2">
-<contactref element="JP1" pad="11"/>
+<contactref element="SV1" pad="11"/>
 </signal>
 </signals>

Commit message: Silk.
Parts:
- moved U$1 6.71 mm to (3.50, 15.0)
Other:
- board text added: "Connect to SHARP GP2Y0A21YK"
Changed lines of the file:
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@@
 <layer number="19" name="Unrouted" color="6" fill="1" visible="yes" active="yes"/>
 <layer number="20" name="Dimension" color="24" fill="1" visible="yes" active="yes"/>
-<layer number="21" name="tPlace" color="7" fill="1" visible="yes" active="yes"/>
-<layer number="22" name="bPlace" color="7" fill="1" visible="no" active="yes"/>
+<layer number="21" name="tPlace" color="7" fill="1" visible="no" active="yes"/>
+<layer number="22" name="bPlace" color="7" fill="1" visible="yes" active="yes"/>
 <layer number="23" name="tOrigins" color="15" fill="1" visible="yes" active="yes"/>
 <layer number="24" name="bOrigins" color="15" fill="1" visible="yes" active="yes"/>
-<layer number="25" name="tNames" color="7" fill="1" visible="yes" active="yes"/>
-<layer number="26" name="bNames" color="7" fill="1" visible="no" active="yes"/>
+<layer number="25" name="tNames" color="7" fill="1" visible="no" active="yes"/>
+<layer number="26" name="bNames" color="7" fill="1" visible="yes" active="yes"/>
 <layer number="27" name="tValues" color="7" fill="1" visible="no" active="yes"/>
 <layer number="28" name="bValues" color="7" fill="1" visible="no" active="yes"/>
@@
 <text x="17.5" y="15.5" size="1" layer="25" rot="R90" align="bottom-center">3P Connertors 0.0.1-X</text>
 <text x="1.5" y="1.5" size="1" layer="25" align="center-left">2-M2.5</text>
+<text x="2.5" y="15" size="1" layer="26" rot="MR90" align="center">Connect to SHARP GP2Y0A21YK</text>
 </plain>
 <attributes>
@@
 <attribute name="VALUE" x="17.445" y="5.34" size="1.27" layer="27" rot="R90"/>
 </element>
-<element name="U$1" library="pineapple" package="PINEAPPLE450_SILK" value="PINEAPPLE450_SILK" x="0.5" y="21" smashed="yes" rot="MR90"/>
+<element name="U$1" library="pineapple" package="PINEAPPLE450_SILK" value="PINEAPPLE450_SILK" x="3.5" y="15" smashed="yes" rot="MR90"/>
 <element name="J31" library="SparkFun-Connectors" library_urn="urn:adsk.eagle:library:513" package="JST-3-PTH" package3d_urn="urn:adsk.eagle:package:38069/1" value="" x="6" y="21" smashed="yes" rot="R90">
 <attribute name="NAME" x="4" y="26" size="1" layer="25" ratio="20" align="center"/>
