File: hardware/peripheral/p2x3p-001.brd (EAGLE design)
At the start: 18 x 31 mm, 7 parts

Commit message: Silk.
Parts:
- moved U$1 0.50 mm to (3.50, 15.5)
Changed lines of the file:
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@@
 <text x="17.5" y="15.5" size="1" layer="25" rot="R90" align="bottom-center">3P Connertors 0.0.1-X</text>
 <text x="1.5" y="1.5" size="1" layer="25" align="center-left">2-M2.5</text>
-<text x="2.5" y="15" size="1" layer="26" rot="MR90" align="center">Connect to SHARP GP2Y0A21YK</text>
+<text x="2.5" y="15.5" size="1" layer="26" rot="MR90" align="center">Connect to SHARP GP2Y0A21YK</text>
 <text x="1" y="23" size="1" layer="25" align="center-left">Vcc</text>
 <text x="1" y="21" size="1" layer="25" align="center-left">GND</text>
@@
 <attribute name="VALUE" x="17.445" y="5.34" size="1.27" layer="27" rot="R90"/>
 </element>
-<element name="U$1" library="pineapple" package="PINEAPPLE450_SILK" value="PINEAPPLE450_SILK" x="3.5" y="15" smashed="yes" rot="MR90"/>
+<element name="U$1" library="pineapple" package="PINEAPPLE450_SILK" value="PINEAPPLE450_SILK" x="3.5" y="15.5" smashed="yes" rot="MR90"/>
 <element name="J31" library="SparkFun-Connectors" library_urn="urn:adsk.eagle:library:513" package="JST-3-PTH" package3d_urn="urn:adsk.eagle:package:38069/1" value="" x="6" y="21" smashed="yes" rot="R90">
 <attribute name="NAME" x="4" y="26" size="1" layer="25" ratio="20" align="center"/>
