File: hardware/peripheral/p2x3p-001.sch (EAGLE design)
At the start: 5 parts

Commit message: WIP.
Parts:
- added C1, C2: (no value), rcl:C-EU025-024X044
Connections:
- net ANLG0: now also J1.1
- net ANLG1: now also J2.1
- net GND: now also C1.2, C2.2, J1.2, J2.2
- net VCC: now also C1.1, C2.1, J1.3, J2.3
Changed lines of the file:
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@@
 <part name="J1" library="SparkFun-Connectors" library_urn="urn:adsk.eagle:library:513" deviceset="CONN_03" device="JST-PTH" package3d_urn="urn:adsk.eagle:package:38069/1"/>
 <part name="J2" library="SparkFun-Connectors" library_urn="urn:adsk.eagle:library:513" deviceset="CONN_03" device="JST-PTH" package3d_urn="urn:adsk.eagle:package:38069/1"/>
+<part name="C1" library="rcl" library_urn="urn:adsk.eagle:library:334" deviceset="C-EU" device="025-024X044" package3d_urn="urn:adsk.eagle:package:23630/1"/>
+<part name="C2" library="rcl" library_urn="urn:adsk.eagle:library:334" deviceset="C-EU" device="025-024X044" package3d_urn="urn:adsk.eagle:package:23630/1"/>
+<part name="SUPPLY2" library="supply2" library_urn="urn:adsk.eagle:library:372" deviceset="GND" device=""/>
+<part name="SUPPLY4" library="supply2" library_urn="urn:adsk.eagle:library:372" deviceset="VCC" device=""/>
 </parts>
 <sheets>
@@
 <attribute name="NAME" x="60.96" y="102.108" size="1.778" layer="95" font="vector"/>
 </instance>
+<instance part="C1" gate="G$1" x="149.86" y="81.28" smashed="yes">
+<attribute name="NAME" x="151.384" y="81.661" size="1.778" layer="95"/>
+<attribute name="VALUE" x="151.384" y="76.581" size="1.778" layer="96"/>
+</instance>
+<instance part="C2" gate="G$1" x="162.56" y="81.28" smashed="yes">
+<attribute name="NAME" x="164.084" y="81.661" size="1.778" layer="95"/>
+<attribute name="VALUE" x="164.084" y="76.581" size="1.778" layer="96"/>
+</instance>
+<instance part="SUPPLY2" gate="GND" x="149.86" y="68.58" smashed="yes">
+<attribute name="VALUE" x="147.955" y="65.405" size="1.778" layer="96"/>
+</instance>
+<instance part="SUPPLY4" gate="G$1" x="149.86" y="93.98" smashed="yes">
+<attribute name="VALUE" x="147.955" y="97.155" size="1.778" layer="96"/>
+</instance>
 </instances>
 <busses>
@@
 <junction x="101.6" y="93.98"/>
 </segment>
+<segment>
+<pinref part="J1" gate="J$1" pin="2"/>
+<wire x1="71.12" y1="109.22" x2="73.66" y2="109.22" width="0.1524" layer="91"/>
+<label x="73.66" y="109.22" size="0.8128" layer="95" xref="yes"/>
+</segment>
+<segment>
+<pinref part="J2" gate="J$1" pin="2"/>
+<wire x1="71.12" y1="96.52" x2="73.66" y2="96.52" width="0.1524" layer="91"/>
+<label x="73.66" y="96.52" size="0.8128" layer="95" xref="yes"/>
+</segment>
+<segment>
+<pinref part="C1" gate="G$1" pin="2"/>
+<wire x1="149.86" y1="76.2" x2="149.86" y2="73.66" width="0.1524" layer="91"/>
+<wire x1="149.86" y1="73.66" x2="162.56" y2="73.66" width="0.1524" layer="91"/>
+<pinref part="C2" gate="G$1" pin="2"/>
+<wire x1="162.56" y1="73.66" x2="162.56" y2="76.2" width="0.1524" layer="91"/>
+<wire x1="149.86" y1="73.66" x2="149.86" y2="71.12" width="0.1524" layer="91"/>
+<junction x="149.86" y="73.66"/>
+<pinref part="SUPPLY2" gate="GND" pin="GND"/>
+</segment>
 </net>
 <net name="DTCT0" class="0">
@@
 <junction x="124.46" y="101.6"/>
 </segment>
+<segment>
+<pinref part="J1" gate="J$1" pin="3"/>
+<wire x1="71.12" y1="111.76" x2="73.66" y2="111.76" width="0.1524" layer="91"/>
+<label x="73.66" y="111.76" size="0.8128" layer="95" xref="yes"/>
+</segment>
+<segment>
+<pinref part="J2" gate="J$1" pin="3"/>
+<wire x1="71.12" y1="99.06" x2="73.66" y2="99.06" width="0.1524" layer="91"/>
+<label x="73.66" y="99.06" size="0.8128" layer="95" xref="yes"/>
+</segment>
+<segment>
+<pinref part="C1" gate="G$1" pin="1"/>
+<wire x1="149.86" y1="83.82" x2="149.86" y2="86.36" width="0.1524" layer="91"/>
+<wire x1="149.86" y1="86.36" x2="162.56" y2="86.36" width="0.1524" layer="91"/>
+<pinref part="C2" gate="G$1" pin="1"/>
+<wire x1="162.56" y1="86.36" x2="162.56" y2="83.82" width="0.1524" layer="91"/>
+<wire x1="149.86" y1="86.36" x2="149.86" y2="91.44" width="0.1524" layer="91"/>
+<junction x="149.86" y="86.36"/>
+<pinref part="SUPPLY4" gate="G$1" pin="VCC"/>
+</segment>
 </net>
 <net name="DTCT1" class="0">
@@
 <label x="96.52" y="106.68" size="0.8128" layer="95" rot="R180" xref="yes"/>
 </segment>
+<segment>
+<pinref part="J1" gate="J$1" pin="1"/>
+<wire x1="71.12" y1="106.68" x2="73.66" y2="106.68" width="0.1524" layer="91"/>
+<label x="73.66" y="106.68" size="0.8128" layer="95" xref="yes"/>
+</segment>
 </net>
 <net name="ANLG1" class="0">
@@
 <wire x1="109.22" y1="101.6" x2="96.52" y2="101.6" width="0.1524" layer="91"/>
 <label x="96.52" y="101.6" size="0.8128" layer="95" rot="R180" xref="yes"/>
+</segment>
+<segment>
+<pinref part="J2" gate="J$1" pin="1"/>
+<wire x1="71.12" y1="93.98" x2="73.66" y2="93.98" width="0.1524" layer="91"/>
+<label x="73.66" y="93.98" size="0.8128" layer="95" xref="yes"/>
 </segment>
 </net>
@@
 packages will not be understood (or retained) with this version.
 </note>
+<note version="8.4" severity="warning">
+Since Version 8.4, EAGLE supports properties for SPICE simulation.
+Probes in schematics and SPICE mapping objects found in parts and library devices
+will not be understood with this version. Update EAGLE to the latest version
+for full support of SPICE simulation.
+</note>
 </compatibility>
