File: hardware/peripheral/p2x3p-001.sch (EAGLE design)
At the start: 7 parts

Commit message: Silk.
Parts:
- renumbered J1 to J31, J2 to J32, JP1 to SV1
Changed lines of the file:
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@@
 <part name="FRAME1" library="frames" library_urn="urn:adsk.eagle:library:229" deviceset="A4L-LOC" device=""/>
 <part name="LOGO1" library="SparkFun-Aesthetics" deviceset="OSHW-LOGO" device="S-COPPER" value="OSHW-LOGOS-COPPER"/>
-<part name="JP1" library="pinhead" library_urn="urn:adsk.eagle:library:325" deviceset="PINHD-2X8" device="" package3d_urn="urn:adsk.eagle:package:22481/2"/>
+<part name="SV1" library="pinhead" library_urn="urn:adsk.eagle:library:325" deviceset="PINHD-2X8" device="" package3d_urn="urn:adsk.eagle:package:22481/2"/>
 <part name="SUPPLY1" library="supply2" library_urn="urn:adsk.eagle:library:372" deviceset="GND" device=""/>
 <part name="SUPPLY3" library="supply2" library_urn="urn:adsk.eagle:library:372" deviceset="VCC" device=""/>
 <part name="U$1" library="pineapple" deviceset="PINEAPPLE450_SILK" device=""/>
-<part name="J1" library="SparkFun-Connectors" library_urn="urn:adsk.eagle:library:513" deviceset="CONN_03" device="JST-PTH" package3d_urn="urn:adsk.eagle:package:38069/1"/>
-<part name="J2" library="SparkFun-Connectors" library_urn="urn:adsk.eagle:library:513" deviceset="CONN_03" device="JST-PTH" package3d_urn="urn:adsk.eagle:package:38069/1"/>
+<part name="J31" library="SparkFun-Connectors" library_urn="urn:adsk.eagle:library:513" deviceset="CONN_03" device="JST-PTH" package3d_urn="urn:adsk.eagle:package:38069/1"/>
+<part name="J32" library="SparkFun-Connectors" library_urn="urn:adsk.eagle:library:513" deviceset="CONN_03" device="JST-PTH" package3d_urn="urn:adsk.eagle:package:38069/1"/>
 <part name="C1" library="rcl" library_urn="urn:adsk.eagle:library:334" deviceset="C-EU" device="025-024X044" package3d_urn="urn:adsk.eagle:package:23630/1"/>
 <part name="C2" library="rcl" library_urn="urn:adsk.eagle:library:334" deviceset="C-EU" device="025-024X044" package3d_urn="urn:adsk.eagle:package:23630/1"/>
@@
 </instance>
 <instance part="LOGO1" gate="G$1" x="241.3" y="165.1" smashed="yes"/>
-<instance part="JP1" gate="A" x="111.76" y="101.6" smashed="yes">
+<instance part="SV1" gate="A" x="111.76" y="101.6" smashed="yes">
 <attribute name="NAME" x="105.41" y="112.395" size="1.778" layer="95"/>
 <attribute name="VALUE" x="105.41" y="86.36" size="1.778" layer="96"/>
@@
 </instance>
 <instance part="U$1" gate="G$1" x="241.3" y="142.24" smashed="yes"/>
-<instance part="J1" gate="J$1" x="63.5" y="109.22" smashed="yes">
+<instance part="J31" gate="J$1" x="63.5" y="109.22" smashed="yes">
 <attribute name="VALUE" x="60.96" y="101.854" size="1.778" layer="96" font="vector"/>
 <attribute name="NAME" x="60.96" y="114.808" size="1.778" layer="95" font="vector"/>
 </instance>
-<instance part="J2" gate="J$1" x="63.5" y="96.52" smashed="yes">
+<instance part="J32" gate="J$1" x="63.5" y="96.52" smashed="yes">
 <attribute name="VALUE" x="60.96" y="89.154" size="1.778" layer="96" font="vector"/>
 <attribute name="NAME" x="60.96" y="102.108" size="1.778" layer="95" font="vector"/>
@@
 <net name="GND" class="0">
 <segment>
-<pinref part="JP1" gate="A" pin="1"/>
+<pinref part="SV1" gate="A" pin="1"/>
 <wire x1="109.22" y1="109.22" x2="101.6" y2="109.22" width="0.1524" layer="91"/>
 <wire x1="101.6" y1="109.22" x2="101.6" y2="104.14" width="0.1524" layer="91"/>
 <pinref part="SUPPLY1" gate="GND" pin="GND"/>
-<pinref part="JP1" gate="A" pin="5"/>
+<pinref part="SV1" gate="A" pin="5"/>
 <wire x1="101.6" y1="104.14" x2="101.6" y2="99.06" width="0.1524" layer="91"/>
 <wire x1="101.6" y1="99.06" x2="101.6" y2="93.98" width="0.1524" layer="91"/>
@@
 <wire x1="109.22" y1="104.14" x2="101.6" y2="104.14" width="0.1524" layer="91"/>
 <junction x="101.6" y="104.14"/>
-<pinref part="JP1" gate="A" pin="9"/>
+<pinref part="SV1" gate="A" pin="9"/>
 <wire x1="109.22" y1="99.06" x2="101.6" y2="99.06" width="0.1524" layer="91"/>
 <junction x="101.6" y="99.06"/>
-<pinref part="JP1" gate="A" pin="13"/>
+<pinref part="SV1" gate="A" pin="13"/>
 <wire x1="109.22" y1="93.98" x2="101.6" y2="93.98" width="0.1524" layer="91"/>
 <junction x="101.6" y="93.98"/>
 </segment>
 <segment>
-<pinref part="J1" gate="J$1" pin="2"/>
+<pinref part="J31" gate="J$1" pin="2"/>
 <wire x1="71.12" y1="109.22" x2="73.66" y2="109.22" width="0.1524" layer="91"/>
 <label x="73.66" y="109.22" size="0.8128" layer="95" xref="yes"/>
 </segment>
 <segment>
-<pinref part="J2" gate="J$1" pin="2"/>
+<pinref part="J32" gate="J$1" pin="2"/>
 <wire x1="71.12" y1="96.52" x2="73.66" y2="96.52" width="0.1524" layer="91"/>
 <label x="73.66" y="96.52" size="0.8128" layer="95" xref="yes"/>
@@
 <net name="DTCT0" class="0">
 <segment>
-<pinref part="JP1" gate="A" pin="2"/>
+<pinref part="SV1" gate="A" pin="2"/>
 <wire x1="116.84" y1="109.22" x2="132.08" y2="109.22" width="0.1524" layer="91"/>
 <label x="132.08" y="109.22" size="0.8128" layer="95" xref="yes"/>
@@
 <net name="VCC" class="0">
 <segment>
-<pinref part="JP1" gate="A" pin="4"/>
+<pinref part="SV1" gate="A" pin="4"/>
 <wire x1="116.84" y1="106.68" x2="124.46" y2="106.68" width="0.1524" layer="91"/>
 <wire x1="124.46" y1="106.68" x2="124.46" y2="124.46" width="0.1524" layer="91"/>
 <pinref part="SUPPLY3" gate="G$1" pin="VCC"/>
-<pinref part="JP1" gate="A" pin="16"/>
+<pinref part="SV1" gate="A" pin="16"/>
 <wire x1="116.84" y1="91.44" x2="124.46" y2="91.44" width="0.1524" layer="91"/>
 <wire x1="124.46" y1="91.44" x2="124.46" y2="96.52" width="0.1524" layer="91"/>
 <junction x="124.46" y="106.68"/>
-<pinref part="JP1" gate="A" pin="12"/>
+<pinref part="SV1" gate="A" pin="12"/>
 <wire x1="124.46" y1="96.52" x2="124.46" y2="101.6" width="0.1524" layer="91"/>
 <wire x1="124.46" y1="101.6" x2="124.46" y2="106.68" width="0.1524" layer="91"/>
 <wire x1="116.84" y1="96.52" x2="124.46" y2="96.52" width="0.1524" layer="91"/>
 <junction x="124.46" y="96.52"/>
-<pinref part="JP1" gate="A" pin="8"/>
+<pinref part="SV1" gate="A" pin="8"/>
 <wire x1="116.84" y1="101.6" x2="124.46" y2="101.6" width="0.1524" layer="91"/>
 <junction x="124.46" y="101.6"/>
 </segment>
 <segment>
-<pinref part="J1" gate="J$1" pin="3"/>
+<pinref part="J31" gate="J$1" pin="3"/>
 <wire x1="71.12" y1="111.76" x2="73.66" y2="111.76" width="0.1524" layer="91"/>
 <label x="73.66" y="111.76" size="0.8128" layer="95" xref="yes"/>
 </segment>
 <segment>
-<pinref part="J2" gate="J$1" pin="3"/>
+<pinref part="J32" gate="J$1" pin="3"/>
 <wire x1="71.12" y1="99.06" x2="73.66" y2="99.06" width="0.1524" layer="91"/>
 <label x="73.66" y="99.06" size="0.8128" layer="95" xref="yes"/>
@@
 <net name="DTCT1" class="0">
 <segment>
-<pinref part="JP1" gate="A" pin="6"/>
+<pinref part="SV1" gate="A" pin="6"/>
 <wire x1="116.84" y1="104.14" x2="132.08" y2="104.14" width="0.1524" layer="91"/>
 <label x="132.08" y="104.14" size="0.8128" layer="95" xref="yes"/>
@@
 <net name="DTCT2" class="0">
 <segment>
-<pinref part="JP1" gate="A" pin="10"/>
+<pinref part="SV1" gate="A" pin="10"/>
 <wire x1="116.84" y1="99.06" x2="132.08" y2="99.06" width="0.1524" layer="91"/>
 <label x="132.08" y="99.06" size="0.8128" layer="95" xref="yes"/>
@@
 <net name="DTCT3" class="0">
 <segment>
-<pinref part="JP1" gate="A" pin="14"/>
+<pinref part="SV1" gate="A" pin="14"/>
 <wire x1="116.84" y1="93.98" x2="132.08" y2="93.98" width="0.1524" layer="91"/>
 <label x="132.08" y="93.98" size="0.8128" layer="95" xref="yes"/>
@@
 <net name="ANLG0" class="0">
 <segment>
-<pinref part="JP1" gate="A" pin="3"/>
+<pinref part="SV1" gate="A" pin="3"/>
 <wire x1="109.22" y1="106.68" x2="96.52" y2="106.68" width="0.1524" layer="91"/>
 <label x="96.52" y="106.68" size="0.8128" layer="95" rot="R180" xref="yes"/>
 </segment>
 <segment>
-<pinref part="J1" gate="J$1" pin="1"/>
+<pinref part="J31" gate="J$1" pin="1"/>
 <wire x1="71.12" y1="106.68" x2="73.66" y2="106.68" width="0.1524" layer="91"/>
 <label x="73.66" y="106.68" size="0.8128" layer="95" xref="yes"/>
@@
 <net name="ANLG1" class="0">
 <segment>
-<pinref part="JP1" gate="A" pin="7"/>
+<pinref part="SV1" gate="A" pin="7"/>
 <wire x1="109.22" y1="101.6" x2="96.52" y2="101.6" width="0.1524" layer="91"/>
 <label x="96.52" y="101.6" size="0.8128" layer="95" rot="R180" xref="yes"/>
 </segment>
 <segment>
-<pinref part="J2" gate="J$1" pin="1"/>
+<pinref part="J32" gate="J$1" pin="1"/>
 <wire x1="71.12" y1="93.98" x2="73.66" y2="93.98" width="0.1524" layer="91"/>
 <label x="73.66" y="93.98" size="0.8128" layer="95" xref="yes"/>
@@
 <net name="ANLG3" class="0">
 <segment>
-<pinref part="JP1" gate="A" pin="15"/>
+<pinref part="SV1" gate="A" pin="15"/>
 <wire x1="109.22" y1="91.44" x2="96.52" y2="91.44" width="0.1524" layer="91"/>
 <label x="96.52" y="91.44" size="0.8128" layer="95" rot="R180" xref="yes"/>
@@
 <net name="ANLG2" class="0">
 <segment>
-<pinref part="JP1" gate="A" pin="11"/>
+<pinref part="SV1" gate="A" pin="11"/>
 <wire x1="109.22" y1="96.52" x2="96.52" y2="96.52" width="0.1524" layer="91"/>
 <label x="96.52" y="96.52" size="0.8128" layer="95" rot="R180" xref="yes"/>
